Commit message: URDF file updated with links

File: InverseKinematics/niryo_one.urdf (robot description, URDF)
Before this commit: robot niryo_one, 9 links, 8 joints
Links:
- link arm_link: geometry collision mesh filename=package://link_descriptions/stl/arm_link.stl; visual mesh filename=package://link_descriptions/collada/arm_link.dae
- link base_link: geometry collision mesh filename=package://link_descriptions/stl/base_link.stl; visual mesh filename=package://link_descriptions/collada/base_link.dae
- link elbow_link: geometry collision mesh filename=package://link_descriptions/stl/elbow_link.stl; visual mesh filename=package://link_descriptions/collada/elbow_link.dae
- link forearm_link: geometry collision mesh filename=package://link_descriptions/stl/forearm_link.stl; visual mesh filename=package://link_descriptions/collada/forearm_link.dae
- link hand_link: geometry collision mesh filename=package://link_descriptions/stl/hand_link.stl; visual mesh filename=package://link_descriptions/collada/hand_link.dae
- link shoulder_link: geometry collision mesh filename=package://link_descriptions/stl/shoulder_link.stl; visual mesh filename=package://link_descriptions/collada/shoulder_link.dae
- link wrist_link: geometry collision mesh filename=package://link_descriptions/stl/wrist_link.stl; visual mesh filename=package://link_descriptions/collada/wrist_link.dae
